Commit message: add retargeting

File: rsc/xarm6/xarm6_allegro_wrist_mounted_rotate copy.urdf (robot description, URDF)
Before this commit: robot xarm6, 29 links, 28 joints
Joints:
- joint joint1: limit lower=-6.28318530718 upper=6.28318530718 effort=500.0 velocity=3.14 -> lower=-6.28318530718 upper=6.28318530718 effort=50.0 velocity=3.14
