Commit message: backup

File: dex_robot/rsc/hands/allegro_hand/allegro_hand_right_free.urdf (robot description, URDF)
Before this commit: robot allegro_right, 29 links, 28 joints
Links:
- removed link link_0.0
- removed link link_1.0
- removed link link_10.0
- removed link link_11.0
- removed link link_11.0_tip
- removed link link_12.0
- removed link link_13.0
- removed link link_14.0
- removed link link_15.0
- removed link link_15.0_tip
- removed link link_2.0
- removed link link_3.0
- removed link link_3.0_tip
- removed link link_4.0
- removed link link_5.0
- removed link link_6.0
- removed link link_7.0
- removed link link_7.0_tip
- removed link link_8.0
- removed link link_9.0
- added link index_base, mass 0.0114; collision mesh filename=meshes/allegro/primary_base.STL; visual mesh filename=meshes/allegro/primary_base.STL
- added link index_distal, mass 0.0094; collision mesh filename=meshes/allegro/primary_distal.STL; visual mesh filename=meshes/allegro/primary_distal.STL
- added link index_medial, mass 0.0376; collision mesh filename=meshes/allegro/primary_medial.STL; visual mesh filename=meshes/allegro/primary_medial.STL
- added link index_proximal, mass 0.0712; collision mesh filename=meshes/allegro/primary_proximal.STL; visual mesh filename=meshes/allegro/primary_proximal.STL
- added link index_tip, mass 0.0166; collision sphere radius=0.015; visual mesh filename=meshes/allegro/primary_tip.STL
- added link middle_base, mass 0.0114; collision mesh filename=meshes/allegro/primary_base.STL; visual mesh filename=meshes/allegro/primary_base.STL
- added link middle_distal, mass 0.0094; collision mesh filename=meshes/allegro/primary_distal.STL; visual mesh filename=meshes/allegro/primary_distal.STL
- added link middle_medial, mass 0.0376; collision mesh filename=meshes/allegro/primary_medial.STL; visual mesh filename=meshes/allegro/primary_medial.STL
- added link middle_proximal, mass 0.0712; collision mesh filename=meshes/allegro/primary_proximal.STL; visual mesh filename=meshes/allegro/primary_proximal.STL
- added link middle_tip, mass 0.0166; collision sphere radius=0.015; visual mesh filename=meshes/allegro/primary_tip.STL
- added link ring_base, mass 0.0114; collision mesh filename=meshes/allegro/primary_base.STL; visual mesh filename=meshes/allegro/primary_base.STL
- added link ring_distal, mass 0.0094; collision mesh filename=meshes/allegro/primary_distal.STL; visual mesh filename=meshes/allegro/primary_distal.STL
- added link ring_medial, mass 0.0376; collision mesh filename=meshes/allegro/primary_medial.STL; visual mesh filename=meshes/allegro/primary_medial.STL
- added link ring_proximal, mass 0.0712; collision mesh filename=meshes/allegro/primary_proximal.STL; visual mesh filename=meshes/allegro/primary_proximal.STL
- added link ring_tip, mass 0.0166; collision sphere radius=0.015; visual mesh filename=meshes/allegro/primary_tip.STL
- added link thumb_base, mass 0.0798; collision mesh filename=meshes/allegro/thumb_base.STL; visual mesh filename=meshes/allegro/thumb_base.STL
- added link thumb_distal, mass 0.0408; collision mesh filename=meshes/allegro/thumb_distal.STL; visual mesh filename=meshes/allegro/thumb_distal.STL
- added link thumb_medial, mass 0.0402; collision mesh filename=meshes/allegro/thumb_medial.STL; visual mesh filename=meshes/allegro/thumb_medial.STL
- added link thumb_proximal, mass 0.0114; collision mesh filename=meshes/allegro/thumb_proximal.STL; visual mesh filename=meshes/allegro/thumb_proximal.STL
- added link thumb_tip, mass 0.0166; collision sphere radius=0.0145; visual mesh filename=meshes/allegro/thumb_tip.STL
Joints:
- removed joint joint_0.0
- removed joint joint_1.0
- removed joint joint_10.0
- removed joint joint_11.0
- removed joint joint_11.0_tip
- removed joint joint_12.0
- removed joint joint_13.0
- removed joint joint_14.0
- removed joint joint_15.0
- removed joint joint_15.0_tip
- removed joint joint_2.0
- removed joint joint_3.0
- removed joint joint_3.0_tip
- removed joint joint_4.0
- removed joint joint_5.0
- removed joint joint_6.0
- removed joint joint_7.0
- removed joint joint_7.0_tip
- removed joint joint_8.0
- removed joint joint_9.0
- added joint index_base: type revolute, parent base_link, child index_base, origin xyz=0 0.0435 -0.001542 rpy=-0.08726646255 0 0, axis 0 0 1, limit lower=-0.57 upper=0.57 effort=15 velocity=7
- added joint index_distal: type revolute, parent index_medial, child index_distal, origin xyz=0 0 0.0384, axis 0 1 0, limit lower=-0.327 upper=1.718 effort=15 velocity=7
- added joint index_medial: type revolute, parent index_proximal, child index_medial, origin xyz=0 0 0.054, axis 0 1 0, limit lower=-0.274 upper=1.809 effort=15 velocity=7
- added joint index_proximal: type revolute, parent index_base, child index_proximal, origin xyz=0 0 0.0164, axis 0 1 0, limit lower=-0.296 upper=1.71 effort=15 velocity=7
- added joint index_tip: type fixed, parent index_distal, child index_tip, origin xyz=0 0 0.0267 rpy=0 0 0
- added joint middle_base: type revolute, parent base_link, child middle_base, axis 0 0 1, limit lower=-0.57 upper=0.57 effort=15 velocity=7
- added joint middle_distal: type revolute, parent middle_medial, child middle_distal, origin xyz=0 0 0.0384, axis 0 1 0, limit lower=-0.327 upper=1.718 effort=15 velocity=7
- added joint middle_medial: type revolute, parent middle_proximal, child middle_medial, origin xyz=0 0 0.054, axis 0 1 0, limit lower=-0.274 upper=1.809 effort=15 velocity=7
- added joint middle_proximal: type revolute, parent middle_base, child middle_proximal, origin xyz=0 0 0.0164, axis 0 1 0, limit lower=-0.296 upper=1.71 effort=15 velocity=7
- added joint middle_tip: type fixed, parent middle_distal, child middle_tip, origin xyz=0 0 0.0267 rpy=0 0 0
- added joint ring_base: type revolute, parent base_link, child ring_base, origin xyz=0 -0.0435 -0.001542 rpy=0.08726646255 0 0, axis 0 0 1, limit lower=-0.57 upper=0.57 effort=15 velocity=7
- added joint ring_distal: type revolute, parent ring_medial, child ring_distal, origin xyz=0 0 0.0384, axis 0 1 0, limit lower=-0.327 upper=1.718 effort=15 velocity=7
- added joint ring_medial: type revolute, parent ring_proximal, child ring_medial, origin xyz=0 0 0.054, axis 0 1 0, limit lower=-0.274 upper=1.809 effort=15 velocity=7
- added joint ring_proximal: type revolute, parent ring_base, child ring_proximal, origin xyz=0 0 0.0164, axis 0 1 0, limit lower=-0.296 upper=1.71 effort=15 velocity=7
- added joint ring_tip: type fixed, parent ring_distal, child ring_tip, origin xyz=0 0 0.0267 rpy=0 0 0
- added joint thumb_base: type revolute, parent base_link, child thumb_base, origin xyz=-0.0182 0.019333 -0.045987 rpy=0 -1.65806278845 -1.5707963259, axis -1 0 0, limit lower=0.36 upper=1.496 effort=15 velocity=7
- added joint thumb_distal: type revolute, parent thumb_medial, child thumb_distal, origin xyz=0 0 0.0514, axis 0 1 0, limit lower=-0.26 upper=1.819 effort=15 velocity=7
- added joint thumb_medial: type revolute, parent thumb_proximal, child thumb_medial, origin xyz=0 0 0.0177, axis 0 1 0, limit lower=-0.289 upper=1.744 effort=15 velocity=7
- added joint thumb_proximal: type revolute, parent thumb_base, child thumb_proximal, origin xyz=-0.027 0.005 0.0399, axis 0 0 1, limit lower=-0.204 upper=1.263 effort=15 velocity=7
- added joint thumb_tip: type fixed, parent thumb_distal, child thumb_tip, origin xyz=0 0 0.0423 rpy=0 0 0
