Commit message: robot controller, clean up src code add lots of ios, teleoperation, starting hand-eyecalibration

File: dex_robot/rsc/xarm6/allegro.urdf (robot description, URDF)
Before this commit: robot xarm6, 28 links, 27 joints
Joints:
- joint world_joint: origin xyz=1 1 1 rpy=0 0 0 -> xyz=0 0 0 rpy=0 0 0
