Commit message: asdf

File: rsc/allegro/allegro_contact.urdf (robot description, URDF)
Before this commit: robot xarm6, 31 links, 30 joints
Links:
- link contact_sensor1: geometry visual mesh filename=meshes/contact_palm.obj
- link contact_sensor2: geometry visual mesh filename=meshes/contact_palm.obj
- link contact_sensor3: geometry visual mesh filename=meshes/contact_palm.obj
- link index_base: geometry collision mesh filename=meshes/primary_base.STL; visual mesh filename=meshes/primary_base.STL
- link index_distal: geometry collision mesh filename=meshes/primary_distal.STL; visual mesh filename=meshes/primary_distal.STL
- link index_medial: geometry collision mesh filename=meshes/primary_medial.STL; visual mesh filename=meshes/primary_medial.STL
- link index_proximal: geometry collision mesh filename=meshes/primary_proximal.STL; visual mesh filename=meshes/primary_proximal.STL
- link index_tip: geometry collision sphere radius=0.015; visual mesh filename=meshes/primary_tip.STL
- link middle_base: geometry collision mesh filename=meshes/primary_base.STL; visual mesh filename=meshes/primary_base.STL
- link middle_distal: geometry collision mesh filename=meshes/primary_distal.STL; visual mesh filename=meshes/primary_distal.STL
- link middle_medial: geometry collision mesh filename=meshes/primary_medial.STL; visual mesh filename=meshes/primary_medial.STL
- link middle_proximal: geometry collision mesh filename=meshes/primary_proximal.STL; visual mesh filename=meshes/primary_proximal.STL
- link middle_tip: geometry collision sphere radius=0.015; visual mesh filename=meshes/primary_tip.STL
- link palm_link: geometry collision mesh filename=meshes/palm_link.obj; visual mesh filename=meshes/palm_link.obj
- link ring_base: geometry collision mesh filename=meshes/primary_base.STL; visual mesh filename=meshes/primary_base.STL
- link ring_distal: geometry collision mesh filename=meshes/primary_distal.STL; visual mesh filename=meshes/primary_distal.STL
- link ring_medial: geometry collision mesh filename=meshes/primary_medial.STL; visual mesh filename=meshes/primary_medial.STL
- link ring_proximal: geometry collision mesh filename=meshes/primary_proximal.STL; visual mesh filename=meshes/primary_proximal.STL
- link ring_tip: geometry collision sphere radius=0.015; visual mesh filename=meshes/primary_tip.STL
- link thumb_base: geometry collision mesh filename=meshes/thumb_base.STL; visual mesh filename=meshes/thumb_base.STL
- link thumb_distal: geometry collision mesh filename=meshes/thumb_distal.STL; visual mesh filename=meshes/thumb_distal.STL
- link thumb_medial: geometry collision mesh filename=meshes/thumb_medial.STL; visual mesh filename=meshes/thumb_medial.STL
- link thumb_proximal: geometry collision mesh filename=meshes/thumb_proximal.STL; visual mesh filename=meshes/thumb_proximal.STL
- link thumb_tip: geometry collision sphere radius=0.0145; visual mesh filename=meshes/thumb_tip.STL

File: rsc/xarm6/allegro_contact.urdf (robot description, URDF)
Before this commit: robot xarm6, 29 links, 28 joints
Links:
- removed link link1
- removed link link2
- removed link link3
- removed link link4
- removed link link5
- removed link link6
- removed link link_base
- added link allegro_root0, mass 4.00000
- added link allegro_root1, mass 0.05
- added link allegro_root2, mass 0.05
- added link allegro_root3, mass 0.05
- added link allegro_root4, mass 0.05
- added link allegro_root5, mass 0.05
- added link contact_sensor1, mass 0.0001; visual mesh filename=meshes/contact/palm.obj
- added link contact_sensor2, mass 0.0001; visual mesh filename=meshes/contact/palm.obj
- added link contact_sensor3, mass 0.0001; visual mesh filename=meshes/contact/palm.obj
- link index_tip: geometry collision sphere radius=0.015; visual mesh filename=meshes/allegro/primary_tip.STL
- link middle_tip: geometry collision sphere radius=0.015; visual mesh filename=meshes/allegro/primary_tip.STL
- link ring_tip: geometry collision sphere radius=0.015; visual mesh filename=meshes/allegro/primary_tip.STL
- link thumb_tip: geometry collision sphere radius=0.0145; visual mesh filename=meshes/allegro/thumb_tip.STL
Joints:
- removed joint gripper_base_joint
- removed joint joint1
- removed joint joint2
- removed joint joint3
- removed joint joint4
- removed joint joint5
- removed joint joint6
- added joint contact_sensor1_attach: type fixed, parent palm_link, child contact_sensor1, origin xyz=0 0 0.0423 rpy=0 0 0
- added joint contact_sensor2_attach: type fixed, parent palm_link, child contact_sensor2, origin xyz=0 0 0.0423 rpy=0 0 0
- added joint contact_sensor3_attach: type fixed, parent palm_link, child contact_sensor3, origin xyz=0 0 0.0423 rpy=0 0 0
- added joint x_joint: type prismatic, parent allegro_root0, child allegro_root1, axis 1 0 0, limit lower=-50.0 upper=50.0 effort=100 velocity=20
- added joint x_rotation_joint: type revolute, parent allegro_root3, child allegro_root4, axis 1 0 0, limit lower=-6.28 upper=6.28 effort=100 velocity=20
- added joint y_joint: type prismatic, parent allegro_root1, child allegro_root2, axis 0 1 0, limit lower=-50.0 upper=50.0 effort=100 velocity=20
- added joint y_rotation_joint: type revolute, parent allegro_root4, child allegro_root5, axis 0 1 0, limit lower=-6.28 upper=6.28 effort=100 velocity=20
- added joint z_joint: type prismatic, parent allegro_root2, child allegro_root3, axis 0 0 1, limit lower=-50.0 upper=50.0 effort=100 velocity=20
- added joint z_rotation_joint: type revolute, parent allegro_root5, child palm_link, axis 0 0 1, limit lower=-6.28 upper=6.28 effort=100 velocity=20
- joint index_tip: origin xyz=0 0 0.0157 rpy=0 -1.570796 0 -> xyz=0 0 0.0267 rpy=0 0 0
- joint middle_tip: origin xyz=0 0 0.0157 rpy=0 -1.570796 0 -> xyz=0 0 0.0267 rpy=0 0 0
- joint ring_tip: origin xyz=0 0 0.0157 rpy=0 -1.570796 0 -> xyz=0 0 0.0267 rpy=0 0 0
- joint thumb_tip: origin xyz=0 0 0.0313 rpy=0 -1.570796 0 -> xyz=0 0 0.0423 rpy=0 0 0
- joint world_joint: child link_base -> allegro_root0

File: rsc/xarm6/xarm6_allegro_wrist_mounted_rotate copy.urdf (robot description, URDF)
Before this commit: robot xarm6, 29 links, 28 joints
Joints:
- joint gripper_base_joint: origin xyz=0 0.035 0.055 rpy=0 -1.57 -1.57 -> xyz=0 0.045 0.045 rpy=0 -1.57 -1.57
- joint index_tip: origin xyz=0 0 0.0157 rpy=0 -1.570796 0 -> xyz=0 0 0.0267 rpy=0 0 0
- joint middle_tip: origin xyz=0 0 0.0157 rpy=0 -1.570796 0 -> xyz=0 0 0.0267 rpy=0 0 0
- joint ring_tip: origin xyz=0 0 0.0157 rpy=0 -1.570796 0 -> xyz=0 0 0.0267 rpy=0 0 0
- joint thumb_tip: origin xyz=0 0 0.0313 rpy=0 -1.570796 0 -> xyz=0 0 0.0423 rpy=0 0 0
